Commit message: Update

File: urdf/amr.urdf.xacro (robot description, xacro)
@@ -20,5 +20,5 @@
         <parent link="base_footprint"/> <!-- 连接到 base_footprint -->
         <child link="base_link"/> <!-- base_link 作为子链接 -->
-        <origin xyz="0 0 0" rpy="0 0 0"/> <!-- 原点和旋转设置，保持位置和方向不变 -->
+        <origin xyz="0 0 0.02" rpy="0 0 0"/> <!-- 原点和旋转设置，保持位置和方向不变 -->
     </joint>
     <!-- 底盘 (base_link) -->
@@ -75,5 +75,5 @@
         <parent link="base_link" />
         <child link="left_wheel" />
-        <origin xyz="0 0 0"/> <!-- 根据底盘和轮子尺寸设置左轮的位置和离地距离 -->
+        <origin xyz="0 0.23215 0.09"/> <!-- 根据底盘和轮子尺寸设置左轮的位置和离地距离 -->
         <axis xyz="0 1 0" /> <!-- 左轮沿 y 轴旋转 -->
     </joint>
@@ -92,5 +92,5 @@
         <parent link="base_link" />
         <child link="right_wheel" />
-        <origin xyz="0 0 0"/>
+        <origin xyz="0 -0.23215 0.09"/>
         <axis xyz="0 1 0" /> <!-- 右轮沿 y 轴旋转 -->
     </joint>
@@ -107,5 +107,5 @@
                 <mesh filename="package://amr_description/meshes/front_caster.stl" scale="${stl_scale}"/>
             </geometry>
-            <origin xyz="0 0 0" rpy="0 0 0" /> <!-- 放置在底盘前方 -->
+            <origin xyz="0 0 0" rpy="0 0 0" />
             <material name="black">
                 <color rgba="${caster_color}"/> <!-- 设置前万向轮的颜色 -->
@@ -116,5 +116,5 @@
         <parent link="base_link" />
         <child link="front_caster" />
-        <origin xyz="0 0 0"/> <!-- 前万向轮放置在底盘前部，离地适中 -->
+        <origin xyz="0.264 0 0.0399"/> <!-- 前万向轮放置在底盘前部，离地适中 -->
         <axis xyz="0 0 1"/> <!-- 前万向轮自由旋转 -->
     </joint>
@@ -124,5 +124,5 @@
                 <mesh filename="package://amr_description/meshes/back_caster.stl" scale="${stl_scale}"/>
             </geometry>
-            <origin xyz="0 0 0" rpy="0 0 0"/> <!-- 放置在底盘后方 -->
+            <origin xyz="0 0 0" rpy="0 0 0"/>
             <material name="black">
                 <color rgba="${caster_color}"/> <!-- 设置后万向轮的颜色 -->
@@ -133,5 +133,5 @@
         <parent link="base_link" />
         <child link="back_caster" />
-        <origin xyz="0 0 0"/> <!-- 后万向轮放置在底盘后部，对称于前万向轮 -->
+        <origin xyz="-0.264 0 0.0399"/> <!-- 后万向轮放置在底盘后部，对称于前万向轮 -->
         <axis xyz="0 0 1"/> <!-- 后万向轮自由旋转 -->
     </joint>
@@ -157,5 +157,5 @@
         <parent link="base_link"/>
         <child link="lidar_link"/>
-        <origin xyz="0 0 0" rpy="0 0 0"/>
+        <origin xyz="0.2815 0 0.144" rpy="0 0 0"/>
     </joint>
 </robot>

Commit message: Update

File: urdf/amr.urdf.xacro (robot description, xacro)
@@ -71,4 +71,10 @@
             </material>
         </visual>
+        <collision>
+            <origin xyz="0 0 0" rpy="0 0 0"/>
+            <geometry>
+                <mesh filename="package://amr_description/meshes/left_wheel.stl" scale="${stl_scale}"/>
+            </geometry>
+        </collision>
     </link>
     <joint name="base_link_to_left_wheel" type="continuous"> <!-- 关节类型为 continuous 表示连续旋转 -->
@@ -88,4 +94,10 @@
             </material>
         </visual>
+        <collision>
+            <origin xyz="0 0 0" rpy="0 0 0"/>
+            <geometry>
+                <mesh filename="package://amr_description/meshes/right_wheel.stl" scale="${stl_scale}"/>
+            </geometry>
+        </collision>
     </link>
     <joint name="base_link_to_right_wheel" type="continuous">
@@ -95,4 +107,58 @@
         <axis xyz="0 1 0" /> <!-- 右轮沿 y 轴旋转 -->
     </joint>
+    <!-- 前后万向轮叉架 -->
+    <link name="front_fork">
+        <visual>
+            <origin xyz="0 0 0" rpy="0 0 0"/> <!-- 叉架的中心位置 -->
+                <geometry>
+                    <mesh filename="package://amr_description/meshes/front_fork.stl" scale="${stl_scale}"/>
+                </geometry>
+            <material name="grey"/>
+        </visual>
+        <collision>
+            <origin xyz="0 0 0" rpy="0 0 0"/>
+            <geometry>
+                <mesh filename="package://amr_description/meshes/front_fork.stl" scale="${stl_scale}"/>
+            </geometry>
+        </collision>
+        <inertial>
+            <mass value="0.5"/> <!-- 叉架的质量 -->
+            <origin xyz="0 0 0" rpy="0 0 0"/>
+            <inertia ixx="0.002" iyy="0.002" izz="0.002" ixy="0" ixz="0" iyz="0"/>
+        </inertial>
+    </link>
+    <!-- 万向节的 joint -->
+    <joint name="base_link_to_front_fork" type="continuous">
+        <parent link="base_link"/> <!-- 父链接为车体 -->
+        <child link="front_fork"/> <!-- 子链接为叉架 -->
+        <origin xyz="0.264 0 0.0399" rpy="0 0 0"/> <!-- 叉架相对于车体的原点和姿态 -->
+        <axis xyz="0 0 1"/> <!-- 允许叉架围绕 Z 轴自由旋转（万向功能） -->
+    </joint>
+    <link name="back_fork">
+        <visual>
+            <origin xyz="0 0 0" rpy="0 0 0"/> <!-- 叉架的中心位置 -->
+                <geometry>
+                    <mesh filename="package://amr_description/meshes/back_fork.stl" scale="${stl_scale}"/>
+                </geometry>
+            <material name="grey"/>
+        </visual>
+        <collision>
+            <origin xyz="0 0 0" rpy="0 0 0"/>
+            <geometry>
+                <mesh filename="package://amr_description/meshes/back_fork.stl" scale="${stl_scale}"/>
+            </geometry>
+        </collision>
+        <inertial>
+            <mass value="0.5"/> <!-- 叉架的质量 -->
+            <origin xyz="0 0 0" rpy="0 0 0"/>
+            <inertia ixx="0.002" iyy="0.002" izz="0.002" ixy="0" ixz="0" iyz="0"/>
+        </inertial>
+    </link>
+    <joint name="base_link_to_back_fork" type="continuous">
+        <parent link="base_link"/> <!-- 父链接为车体 -->
+        <child link="back_fork"/> <!-- 子链接为叉架 -->
+        <origin xyz="-0.264 0 0.0399" rpy="0 0 0"/> <!-- 叉架相对于车体的原点和姿态 -->
+        <axis xyz="0 0 1"/> <!-- 允许叉架围绕 Z 轴自由旋转（万向功能） -->
+    </joint>
     <!-- 前后万向轮 (支撑轮) -->
     <!--
@@ -112,10 +178,16 @@
             </material>
         </visual>
-    </link>
-    <joint name="base_link_to_front_caster" type="continuous">
-        <parent link="base_link" />
+        <collision>
+            <origin xyz="0 0 0" rpy="0 0 0"/>
+            <geometry>
+                <mesh filename="package://amr_description/meshes/front_caster.stl" scale="${stl_scale}"/>
+            </geometry>
+        </collision>
+    </link>
+    <joint name="front_fork_to_front_caster" type="continuous">
+        <parent link="front_fork" />
         <child link="front_caster" />
-        <origin xyz="0.264 0 0.0399"/> <!-- 前万向轮放置在底盘前部，离地适中 -->
-        <axis xyz="0 0 1"/> <!-- 前万向轮自由旋转 -->
+        <origin xyz="0.252 0 0.016"/> <!-- 前万向轮放置在底盘前部，离地适中 -->
+        <axis xyz="0 1 0"/> <!-- 前万向轮自由旋转 -->
     </joint>
     <link name="back_caster">
@@ -129,10 +201,16 @@
             </material>
         </visual>
-    </link>
-    <joint name="base_link_to_back_caster" type="continuous">
-        <parent link="base_link" />
+        <collision>
+            <origin xyz="0 0 0" rpy="0 0 0"/>
+            <geometry>
+                <mesh filename="package://amr_description/meshes/back_caster.stl" scale="${stl_scale}"/>
+            </geometry>
+        </collision>
+    </link>
+    <joint name="back_fork_to_back_caster" type="continuous">
+        <parent link="back_fork" />
         <child link="back_caster" />
-        <origin xyz="-0.264 0 0.0399"/> <!-- 后万向轮放置在底盘后部，对称于前万向轮 -->
-        <axis xyz="0 0 1"/> <!-- 后万向轮自由旋转 -->
+        <origin xyz="-0.276 0 0.016"/> <!-- 后万向轮放置在底盘后部，对称于前万向轮 -->
+        <axis xyz="0 1 0"/> <!-- 后万向轮自由旋转 -->
     </joint>
     <!-- 激光雷达 (lidar_link) -->
@@ -152,4 +230,10 @@
             </material>
         </visual>
+        <collision>
+            <origin xyz="0 0 0" rpy="0 0 0"/>
+            <geometry>
+                <mesh filename="package://amr_description/meshes/lidar_link.stl" scale="${stl_scale}"/>
+            </geometry>
+        </collision>
     </link>
     <!-- lidar_link 通过固定关节连接到 base_link -->

Commit message: Update

File: urdf/amr.urdf.xacro (robot description, xacro)
@@ -188,5 +188,5 @@
         <parent link="front_fork" />
         <child link="front_caster" />
-        <origin xyz="0.252 0 0.016"/> <!-- 前万向轮放置在底盘前部，离地适中 -->
+        <origin xyz="-0.012 0 -0.0239"/> <!-- 前万向轮放置在底盘前部，离地适中 -->
         <axis xyz="0 1 0"/> <!-- 前万向轮自由旋转 -->
     </joint>
@@ -211,5 +211,5 @@
         <parent link="back_fork" />
         <child link="back_caster" />
-        <origin xyz="-0.276 0 0.016"/> <!-- 后万向轮放置在底盘后部，对称于前万向轮 -->
+        <origin xyz="-0.012 0 -0.0239"/> <!-- 后万向轮放置在底盘后部，对称于前万向轮 -->
         <axis xyz="0 1 0"/> <!-- 后万向轮自由旋转 -->
     </joint>

Commit message: Update

File: urdf/amr.urdf.xacro (robot description, xacro)
@@ -214,15 +214,15 @@
         <axis xyz="0 1 0"/> <!-- 后万向轮自由旋转 -->
     </joint>
-    <!-- 激光雷达 (lidar_link) -->
+    <!-- 激光雷达 (laser) -->
     <!--
         参数说明:
             - 高度: 3.885厘米
             - 半径: 7.7厘米
-            - STL 网格文件: lidar_link.stl
-    -->
-    <link name="lidar_link">
-        <visual>
-            <geometry>
-                <mesh filename="package://amr_description/meshes/lidar_link.stl" scale="${stl_scale}"/>
+            - STL 网格文件: laser.stl
+    -->
+    <link name="laser">
+        <visual>
+            <geometry>
+                <mesh filename="package://amr_description/meshes/laser.stl" scale="${stl_scale}"/>
             </geometry>
             <material name="black">
@@ -233,12 +233,12 @@
             <origin xyz="0 0 0" rpy="0 0 0"/>
             <geometry>
-                <mesh filename="package://amr_description/meshes/lidar_link.stl" scale="${stl_scale}"/>
-            </geometry>
-        </collision>
-    </link>
-    <!-- lidar_link 通过固定关节连接到 base_link -->
-    <joint name="lidar_joint" type="fixed">
+                <mesh filename="package://amr_description/meshes/laser.stl" scale="${stl_scale}"/>
+            </geometry>
+        </collision>
+    </link>
+    <!-- laser 通过固定关节连接到 base_link -->
+    <joint name="base_link_to_laser" type="fixed">
         <parent link="base_link"/>
-        <child link="lidar_link"/>
+        <child link="laser"/>
         <origin xyz="0.2815 0 0.144" rpy="0 0 0"/>
     </joint>

Commit message: Update

File: urdf/amr.urdf.xacro (robot description, xacro)
@@ -14,5 +14,13 @@
     <!-- base_footprint 是虚拟的参考框架，用来定义机器人在地面上的位置和姿态 -->
     <link name="base_footprint">
-        <!-- 可省略visual部分，使其仅作为参考框架 -->
+        <visual>
+            <origin xyz="0 0 0" rpy="0 0 0" />
+            <geometry>
+                <box size="0.05 0.05 0.001" />
+            </geometry>
+            <material name="transparent">
+                <color rgba="0.0 0.0 0.0 0.0"/> <!-- 设置底盘颜色 -->
+            </material>
+        </visual>
     </link>
     <!-- base_link 是底盘的主要框架，与虚拟根链接 base_footprint 通过固定关节连接 -->
@@ -20,5 +28,5 @@
         <parent link="base_footprint"/> <!-- 连接到 base_footprint -->
         <child link="base_link"/> <!-- base_link 作为子链接 -->
-        <origin xyz="0 0 0.02" rpy="0 0 0"/> <!-- 原点和旋转设置，保持位置和方向不变 -->
+        <origin xyz="0 0 0" rpy="0 0 0"/> <!-- 原点和旋转设置，保持位置和方向不变 -->
     </joint>
     <!-- 底盘 (base_link) -->

Commit message: Update

File: urdf/amr.urdf.xacro (robot description, xacro)
@@ -249,5 +249,5 @@
         <parent link="base_link"/>
         <child link="laser"/>
-        <origin xyz="0.2815 0 0.144" rpy="0 0 0"/>
+        <origin xyz="0.2815 0 0.17223265" rpy="0 0 0"/>
     </joint>
 </robot>

Commit message: Update

File: urdf/amr.urdf.xacro (robot description, xacro)
@@ -28,5 +28,5 @@
         <parent link="base_footprint"/> <!-- 连接到 base_footprint -->
         <child link="base_link"/> <!-- base_link 作为子链接 -->
-        <origin xyz="0 0 0" rpy="0 0 0"/> <!-- 原点和旋转设置，保持位置和方向不变 -->
+        <origin xyz="0 0 0.02" rpy="0 0 0"/> <!-- 原点和旋转设置，保持位置和方向不变 -->
     </joint>
     <!-- 底盘 (base_link) -->
@@ -89,5 +89,5 @@
         <parent link="base_link" />
         <child link="left_wheel" />
-        <origin xyz="0 0.23215 0.09"/> <!-- 根据底盘和轮子尺寸设置左轮的位置和离地距离 -->
+        <origin xyz="0 0.23215 0.07"/> <!-- 根据底盘和轮子尺寸设置左轮的位置和离地距离 -->
         <axis xyz="0 1 0" /> <!-- 左轮沿 y 轴旋转 -->
     </joint>
@@ -112,5 +112,5 @@
         <parent link="base_link" />
         <child link="right_wheel" />
-        <origin xyz="0 -0.23215 0.09"/>
+        <origin xyz="0 -0.23215 0.07"/>
         <axis xyz="0 1 0" /> <!-- 右轮沿 y 轴旋转 -->
     </joint>
@@ -140,5 +140,5 @@
         <parent link="base_link"/> <!-- 父链接为车体 -->
         <child link="front_fork"/> <!-- 子链接为叉架 -->
-        <origin xyz="0.264 0 0.0399" rpy="0 0 0"/> <!-- 叉架相对于车体的原点和姿态 -->
+        <origin xyz="0.264 0 0.0169" rpy="0 0 0"/> <!-- 叉架相对于车体的原点和姿态 -->
         <axis xyz="0 0 1"/> <!-- 允许叉架围绕 Z 轴自由旋转（万向功能） -->
     </joint>
@@ -166,5 +166,5 @@
         <parent link="base_link"/> <!-- 父链接为车体 -->
         <child link="back_fork"/> <!-- 子链接为叉架 -->
-        <origin xyz="-0.264 0 0.0399" rpy="0 0 0"/> <!-- 叉架相对于车体的原点和姿态 -->
+        <origin xyz="-0.264 0 0.0169" rpy="0 0 0"/> <!-- 叉架相对于车体的原点和姿态 -->
         <axis xyz="0 0 1"/> <!-- 允许叉架围绕 Z 轴自由旋转（万向功能） -->
     </joint>
@@ -249,5 +249,5 @@
         <parent link="base_link"/>
         <child link="laser"/>
-        <origin xyz="0.2815 0 0.17223265" rpy="0 0 0"/>
+        <origin xyz="0.2815 0 0.15223265" rpy="0 0 0"/>
     </joint>
 </robot>

Commit message: Update

File: urdf/amr.urdf.xacro (robot description, xacro)
@@ -28,5 +28,5 @@
         <parent link="base_footprint"/> <!-- 连接到 base_footprint -->
         <child link="base_link"/> <!-- base_link 作为子链接 -->
-        <origin xyz="0 0 0.02" rpy="0 0 0"/> <!-- 原点和旋转设置，保持位置和方向不变 -->
+        <origin xyz="0 0 0" rpy="0 0 0"/> <!-- 原点和旋转设置，保持位置和方向不变 -->
     </joint>
     <!-- 底盘 (base_link) -->
@@ -89,5 +89,5 @@
         <parent link="base_link" />
         <child link="left_wheel" />
-        <origin xyz="0 0.23215 0.07"/> <!-- 根据底盘和轮子尺寸设置左轮的位置和离地距离 -->
+        <origin xyz="0 0.23215 0.09"/> <!-- 根据底盘和轮子尺寸设置左轮的位置和离地距离 -->
         <axis xyz="0 1 0" /> <!-- 左轮沿 y 轴旋转 -->
     </joint>
@@ -112,5 +112,5 @@
         <parent link="base_link" />
         <child link="right_wheel" />
-        <origin xyz="0 -0.23215 0.07"/>
+        <origin xyz="0 -0.23215 0.09"/>
         <axis xyz="0 1 0" /> <!-- 右轮沿 y 轴旋转 -->
     </joint>
@@ -140,5 +140,5 @@
         <parent link="base_link"/> <!-- 父链接为车体 -->
         <child link="front_fork"/> <!-- 子链接为叉架 -->
-        <origin xyz="0.264 0 0.0169" rpy="0 0 0"/> <!-- 叉架相对于车体的原点和姿态 -->
+        <origin xyz="0.264 0 0.0399" rpy="0 0 0"/> <!-- 叉架相对于车体的原点和姿态 -->
         <axis xyz="0 0 1"/> <!-- 允许叉架围绕 Z 轴自由旋转（万向功能） -->
     </joint>
@@ -166,5 +166,5 @@
         <parent link="base_link"/> <!-- 父链接为车体 -->
         <child link="back_fork"/> <!-- 子链接为叉架 -->
-        <origin xyz="-0.264 0 0.0169" rpy="0 0 0"/> <!-- 叉架相对于车体的原点和姿态 -->
+        <origin xyz="-0.264 0 0.0399" rpy="0 0 0"/> <!-- 叉架相对于车体的原点和姿态 -->
         <axis xyz="0 0 1"/> <!-- 允许叉架围绕 Z 轴自由旋转（万向功能） -->
     </joint>
@@ -249,5 +249,5 @@
         <parent link="base_link"/>
         <child link="laser"/>
-        <origin xyz="0.2815 0 0.15223265" rpy="0 0 0"/>
+        <origin xyz="0.2815 0 0.17223265" rpy="0 0 0"/>
     </joint>
 </robot>

Commit message: Update

File: urdf/amr.urdf.xacro (robot description, xacro)
@@ -25,5 +25,5 @@
     </link>
     <!-- base_link 是底盘的主要框架，与虚拟根链接 base_footprint 通过固定关节连接 -->
-    <joint name="fixed_base" type="fixed">
+    <joint name="base_joint" type="fixed">
         <parent link="base_footprint"/> <!-- 连接到 base_footprint -->
         <child link="base_link"/> <!-- base_link 作为子链接 -->

Commit message: Update

File: urdf/amr.urdf.xacro (robot description, xacro)
@@ -25,5 +25,5 @@
     </link>
     <!-- base_link 是底盘的主要框架，与虚拟根链接 base_footprint 通过固定关节连接 -->
-    <joint name="base_joint" type="fixed">
+    <joint name="base_footprint_to_base_link" type="fixed">
         <parent link="base_footprint"/> <!-- 连接到 base_footprint -->
         <child link="base_link"/> <!-- base_link 作为子链接 -->

Commit message: Update

File: urdf/amr.urdf.xacro (robot description, xacro)
@@ -4,6 +4,4 @@
     <!-- 定义 STL 比例，用于缩放 STL 文件的网格 -->
     <xacro:property name="stl_scale" value="0.001 0.001 0.001"/>
-    <!-- 定义底盘的质量 (kg) -->
-    <xacro:property name="base_link_mass" value="50.0"/>
     <!-- 定义各个部分的颜色: 底盘、驱动轮、万向轮、激光雷达 -->
     <xacro:property name="base_color" value="0.5 0.5 0.5 1.0"/> <!-- 本体的颜色：灰色 -->
@@ -19,7 +17,4 @@
                 <box size="0.05 0.05 0.001" />
             </geometry>
-            <material name="transparent">
-                <color rgba="0.0 0.0 0.0 0.0"/> <!-- 设置底盘颜色 -->
-            </material>
         </visual>
     </link>
@@ -54,9 +49,4 @@
             </geometry>
         </collision>
-        <inertial>
-            <mass value="${base_link_mass}"/> <!-- 定义底盘质量 -->
-            <origin xyz="0 0 0" rpy="0 0 0"/> <!-- 定义惯性原点为零点 -->
-            <inertia ixx="1" iyy="1" izz="1" ixy="0" ixz="0" iyz="0"/> <!-- 简化的惯性张量参数 -->
-        </inertial>
     </link>
     <!-- 左右驱动轮 -->

Commit message: Update

File: urdf/amr.urdf.xacro (robot description, xacro)
@@ -239,5 +239,5 @@
         <parent link="base_link"/>
         <child link="laser"/>
-        <origin xyz="0.2815 0 0.17223265" rpy="0 0 0"/>
+        <origin xyz="0.2815 0 0.17223265" rpy="0 0 3.14159265"/> <!-- 激光雷达相对于车体的原点和姿态 -->
     </joint>
 </robot>

Commit message: Update

File: urdf/amr.urdf.xacro (robot description, xacro)
@@ -23,5 +23,5 @@
         <parent link="base_footprint"/> <!-- 连接到 base_footprint -->
         <child link="base_link"/> <!-- base_link 作为子链接 -->
-        <origin xyz="0 0 0" rpy="0 0 0"/> <!-- 原点和旋转设置，保持位置和方向不变 -->
+        <origin xyz="0 0 0.02" rpy="0 0 0"/> <!-- 原点和旋转设置，保持位置和方向不变 -->
     </joint>
     <!-- 底盘 (base_link) -->
@@ -64,5 +64,4 @@
                 <mesh filename="package://amr_description/meshes/left_wheel.stl" scale="${stl_scale}"/>
             </geometry>
-            <origin xyz="0 0 0" rpy="0 0 0"/> <!-- 车轮的几何模型位于轮轴上 -->
             <material name="red">
                 <color rgba="${wheel_color}"/> <!-- 设置轮子的颜色 -->
@@ -70,5 +69,4 @@
         </visual>
         <collision>
-            <origin xyz="0 0 0" rpy="0 0 0"/>
             <geometry>
                 <mesh filename="package://amr_description/meshes/left_wheel.stl" scale="${stl_scale}"/>
@@ -87,5 +85,4 @@
                 <mesh filename="package://amr_description/meshes/right_wheel.stl" scale="${stl_scale}"/>
             </geometry>
-            <origin xyz="0 0 0" rpy="0 0 0"/>
             <material name="red">
                 <color rgba="${wheel_color}"/> <!-- 颜色设置一致 -->
@@ -93,5 +90,4 @@
         </visual>
         <collision>
-            <origin xyz="0 0 0" rpy="0 0 0"/>
             <geometry>
                 <mesh filename="package://amr_description/meshes/right_wheel.stl" scale="${stl_scale}"/>
@@ -108,21 +104,14 @@
     <link name="front_fork">
         <visual>
-            <origin xyz="0 0 0" rpy="0 0 0"/> <!-- 叉架的中心位置 -->
-                <geometry>
-                    <mesh filename="package://amr_description/meshes/front_fork.stl" scale="${stl_scale}"/>
-                </geometry>
+            <geometry>
+                <mesh filename="package://amr_description/meshes/front_fork.stl" scale="${stl_scale}"/>
+            </geometry>
             <material name="grey"/>
         </visual>
         <collision>
-            <origin xyz="0 0 0" rpy="0 0 0"/>
             <geometry>
                 <mesh filename="package://amr_description/meshes/front_fork.stl" scale="${stl_scale}"/>
             </geometry>
         </collision>
-        <inertial>
-            <mass value="0.5"/> <!-- 叉架的质量 -->
-            <origin xyz="0 0 0" rpy="0 0 0"/>
-            <inertia ixx="0.002" iyy="0.002" izz="0.002" ixy="0" ixz="0" iyz="0"/>
-        </inertial>
     </link>
     <!-- 万向节的 joint -->
@@ -135,21 +124,14 @@
     <link name="back_fork">
         <visual>
-            <origin xyz="0 0 0" rpy="0 0 0"/> <!-- 叉架的中心位置 -->
-                <geometry>
-                    <mesh filename="package://amr_description/meshes/back_fork.stl" scale="${stl_scale}"/>
-                </geometry>
+            <geometry>
+                <mesh filename="package://amr_description/meshes/back_fork.stl" scale="${stl_scale}"/>
+            </geometry>
             <material name="grey"/>
         </visual>
         <collision>
-            <origin xyz="0 0 0" rpy="0 0 0"/>
             <geometry>
                 <mesh filename="package://amr_description/meshes/back_fork.stl" scale="${stl_scale}"/>
             </geometry>
         </collision>
-        <inertial>
-            <mass value="0.5"/> <!-- 叉架的质量 -->
-            <origin xyz="0 0 0" rpy="0 0 0"/>
-            <inertia ixx="0.002" iyy="0.002" izz="0.002" ixy="0" ixz="0" iyz="0"/>
-        </inertial>
     </link>
     <joint name="base_link_to_back_fork" type="continuous">
@@ -171,5 +153,4 @@
                 <mesh filename="package://amr_description/meshes/front_caster.stl" scale="${stl_scale}"/>
             </geometry>
-            <origin xyz="0 0 0" rpy="0 0 0" />
             <material name="black">
                 <color rgba="${caster_color}"/> <!-- 设置前万向轮的颜色 -->
@@ -177,5 +158,4 @@
         </visual>
         <collision>
-            <origin xyz="0 0 0" rpy="0 0 0"/>
             <geometry>
                 <mesh filename="package://amr_description/meshes/front_caster.stl" scale="${stl_scale}"/>
@@ -194,5 +174,4 @@
                 <mesh filename="package://amr_description/meshes/back_caster.stl" scale="${stl_scale}"/>
             </geometry>
-            <origin xyz="0 0 0" rpy="0 0 0"/>
             <material name="black">
                 <color rgba="${caster_color}"/> <!-- 设置后万向轮的颜色 -->
@@ -200,5 +179,4 @@
         </visual>
         <collision>
-            <origin xyz="0 0 0" rpy="0 0 0"/>
             <geometry>
                 <mesh filename="package://amr_description/meshes/back_caster.stl" scale="${stl_scale}"/>
@@ -229,5 +207,4 @@
         </visual>
         <collision>
-            <origin xyz="0 0 0" rpy="0 0 0"/>
             <geometry>
                 <mesh filename="package://amr_description/meshes/laser.stl" scale="${stl_scale}"/>

Commit message: Update

File: urdf/amr.urdf.xacro (robot description, xacro)
@@ -35,4 +35,5 @@
     <link name="base_link">
         <visual>
+            <origin xyz="0 0 0" rpy="0 0 0" />
             <geometry>
                 <!-- 视觉形状 -->

Commit message: Update

File: urdf/amr.urdf.xacro (robot description, xacro)
@@ -23,5 +23,5 @@
         <parent link="base_footprint"/> <!-- 连接到 base_footprint -->
         <child link="base_link"/> <!-- base_link 作为子链接 -->
-        <origin xyz="0 0 0.02" rpy="0 0 0"/> <!-- 原点和旋转设置，保持位置和方向不变 -->
+        <origin xyz="0 0 0" rpy="0 0 0"/> <!-- 原点和旋转设置，保持位置和方向不变 -->
     </joint>
     <!-- 底盘 (base_link) -->
@@ -35,5 +35,5 @@
     <link name="base_link">
         <visual>
-            <origin xyz="0 0 0" rpy="0 0 0" />
+            <origin xyz="0 0 0.02" rpy="0 0 0" />
             <geometry>
                 <!-- 视觉形状 -->
