Commit message: Update

File: urdf/amr.urdf.xacro (robot description, xacro)
@@ -217,5 +217,5 @@
         <parent link="base_link"/>
         <child link="laser"/>
-        <origin xyz="0.2815 0 0.17223265" rpy="0 0 3.14159265"/> <!-- 激光雷达相对于车体的原点和姿态 -->
+        <origin xyz="0.2815 0 0.15223265" rpy="0 0 3.14159265"/> <!-- 激光雷达相对于车体的原点和姿态 -->
     </joint>
 </robot>

Commit message: Update

File: urdf/amr.urdf.xacro (robot description, xacro)
@@ -217,5 +217,5 @@
         <parent link="base_link"/>
         <child link="laser"/>
-        <origin xyz="0.2815 0 0.15223265" rpy="0 0 3.14159265"/> <!-- 激光雷达相对于车体的原点和姿态 -->
+        <origin xyz="0.2815 0 0.17223265" rpy="0 0 3.14159265"/> <!-- 激光雷达相对于车体的原点和姿态 -->
     </joint>
 </robot>

Commit message: Update

File: urdf/amr.urdf.xacro (robot description, xacro)
@@ -217,5 +217,5 @@
         <parent link="base_link"/>
         <child link="laser"/>
-        <origin xyz="0.2815 0 0.17223265" rpy="0 0 3.14159265"/> <!-- 激光雷达相对于车体的原点和姿态 -->
+        <origin xyz="0.2815 0 0.17223265" rpy="0 0 0"/> <!-- 激光雷达相对于车体的原点和姿态 -->
     </joint>
 </robot>

Commit message: Update

File: urdf/amr.urdf.xacro (robot description, xacro)
@@ -217,5 +217,5 @@
         <parent link="base_link"/>
         <child link="laser"/>
-        <origin xyz="0.2815 0 0.17223265" rpy="0 0 0"/> <!-- 激光雷达相对于车体的原点和姿态 -->
+        <origin xyz="0.2815 0 0.17223265" rpy="0 0 3.1415926"/> <!-- 激光雷达相对于车体的原点和姿态 -->
     </joint>
 </robot>

Commit message: Update

File: urdf/amr.urdf.xacro (robot description, xacro)
@@ -217,5 +217,5 @@
         <parent link="base_link"/>
         <child link="laser"/>
-        <origin xyz="0.2815 0 0.17223265" rpy="0 0 3.1415926"/> <!-- 激光雷达相对于车体的原点和姿态 -->
+        <origin xyz="0.2815 0 0.17223265" rpy="0 0 0"/> <!-- 激光雷达相对于车体的原点和姿态 -->
     </joint>
 </robot>

Commit message: Update

File: urdf/amr.urdf.xacro (robot description, xacro)
@@ -217,5 +217,5 @@
         <parent link="base_link"/>
         <child link="laser"/>
-        <origin xyz="0.2815 0 0.17223265" rpy="0 0 0"/> <!-- 激光雷达相对于车体的原点和姿态 -->
+        <origin xyz="0.2815 0 0.17223265" rpy="0 0 -3.1415926"/> <!-- 激光雷达相对于车体的原点和姿态 -->
     </joint>
 </robot>

Commit message: Update

File: urdf/amr.urdf.xacro (robot description, xacro)
@@ -217,5 +217,5 @@
         <parent link="base_link"/>
         <child link="laser"/>
-        <origin xyz="0.2815 0 0.17223265" rpy="0 0 -3.1415926"/> <!-- 激光雷达相对于车体的原点和姿态 -->
+        <origin xyz="0.2815 0 0.17223265" rpy="0 0 0"/> <!-- 激光雷达相对于车体的原点和姿态 -->
     </joint>
 </robot>

Commit message: Update

File: urdf/amr.urdf.xacro (robot description, xacro)
@@ -200,4 +200,5 @@
     <link name="laser">
         <visual>
+            <origin xyz="0 0 0" rpy="0 0 3.1415926"/>
             <geometry>
                 <mesh filename="package://amr_description/meshes/laser.stl" scale="${stl_scale}"/>
@@ -208,4 +209,5 @@
         </visual>
         <collision>
+            <origin xyz="0 0 0" rpy="0 0 3.1415926"/>
             <geometry>
                 <mesh filename="package://amr_description/meshes/laser.stl" scale="${stl_scale}"/>

Commit message: Update

File: urdf/amr.urdf.xacro (robot description, xacro)
@@ -200,5 +200,4 @@
     <link name="laser">
         <visual>
-            <origin xyz="0 0 0" rpy="0 0 3.1415926"/>
             <geometry>
                 <mesh filename="package://amr_description/meshes/laser.stl" scale="${stl_scale}"/>
@@ -209,5 +208,4 @@
         </visual>
         <collision>
-            <origin xyz="0 0 0" rpy="0 0 3.1415926"/>
             <geometry>
                 <mesh filename="package://amr_description/meshes/laser.stl" scale="${stl_scale}"/>

Commit message: Update

File: urdf/amr.urdf.xacro (robot description, xacro)
@@ -217,5 +217,5 @@
         <parent link="base_link"/>
         <child link="laser"/>
-        <origin xyz="0.2815 0 0.17223265" rpy="0 0 0"/> <!-- 激光雷达相对于车体的原点和姿态 -->
+        <origin xyz="0.2815 0 0.17223265" rpy="0 0 ${pi}"/> <!-- 激光雷达相对于车体的原点和姿态 -->
     </joint>
 </robot>

Commit message: Update

File: urdf/amr.urdf.xacro (robot description, xacro)
@@ -23,5 +23,5 @@
         <parent link="base_footprint"/> <!-- 连接到 base_footprint -->
         <child link="base_link"/> <!-- base_link 作为子链接 -->
-        <origin xyz="0 0 0" rpy="0 0 0"/> <!-- 原点和旋转设置，保持位置和方向不变 -->
+        <origin xyz="0 0 0" rpy="0 0 ${pi}"/> <!-- 原点和旋转设置 -->
     </joint>
     <!-- 底盘 (base_link) -->

Commit message: Update

File: urdf/amr.urdf.xacro (robot description, xacro)
@@ -13,5 +13,5 @@
     <link name="base_footprint">
         <visual>
-            <origin xyz="0 0 0" rpy="0 0 0" />
+            <origin xyz="0 0 0" rpy="0 0 ${pi}" />
             <geometry>
                 <box size="0.05 0.05 0.001" />
@@ -23,5 +23,5 @@
         <parent link="base_footprint"/> <!-- 连接到 base_footprint -->
         <child link="base_link"/> <!-- base_link 作为子链接 -->
-        <origin xyz="0 0 0" rpy="0 0 ${pi}"/> <!-- 原点和旋转设置 -->
+        <origin xyz="0 0 0" rpy="0 0 0"/> <!-- 原点和旋转设置 -->
     </joint>
     <!-- 底盘 (base_link) -->

Commit message: Update

File: urdf/amr.urdf.xacro (robot description, xacro)
@@ -13,5 +13,5 @@
     <link name="base_footprint">
         <visual>
-            <origin xyz="0 0 0" rpy="0 0 ${pi}" />
+            <origin xyz="0 0 0" rpy="0 0 0" />
             <geometry>
                 <box size="0.05 0.05 0.001" />
@@ -35,5 +35,5 @@
     <link name="base_link">
         <visual>
-            <origin xyz="0 0 0.02" rpy="0 0 0" />
+            <origin xyz="0 0 0.02" rpy="0 0 ${pi}" />
             <geometry>
                 <!-- 视觉形状 -->

Commit message: Update

File: urdf/amr.urdf.xacro (robot description, xacro)
@@ -217,5 +217,5 @@
         <parent link="base_link"/>
         <child link="laser"/>
-        <origin xyz="0.2815 0 0.17223265" rpy="0 0 ${pi}"/> <!-- 激光雷达相对于车体的原点和姿态 -->
+        <origin xyz="0.2815 0 0.17223265" rpy="0 0 0"/> <!-- 激光雷达相对于车体的原点和姿态 -->
     </joint>
 </robot>

Commit message: Update

File: urdf/amr.urdf.xacro (robot description, xacro)
@@ -35,5 +35,5 @@
     <link name="base_link">
         <visual>
-            <origin xyz="0 0 0.02" rpy="0 0 ${pi}" />
+            <origin xyz="0 0 0.02" rpy="0 0 0" />
             <geometry>
                 <!-- 视觉形状 -->
@@ -217,5 +217,5 @@
         <parent link="base_link"/>
         <child link="laser"/>
-        <origin xyz="0.2815 0 0.17223265" rpy="0 0 0"/> <!-- 激光雷达相对于车体的原点和姿态 -->
+        <origin xyz="0.2815 0 0.17223265" rpy="0 0 ${pi}"/> <!-- 激光雷达相对于车体的原点和姿态 -->
     </joint>
 </robot>

Commit message: Update

File: urdf/amr.urdf.xacro (robot description, xacro)
@@ -217,5 +217,5 @@
         <parent link="base_link"/>
         <child link="laser"/>
-        <origin xyz="0.2815 0 0.17223265" rpy="0 0 ${pi}"/> <!-- 激光雷达相对于车体的原点和姿态 -->
+        <origin xyz="-0.2815 0 0.17223265" rpy="0 0 ${pi}"/> <!-- 激光雷达相对于车体的原点和姿态 -->
     </joint>
 </robot>

Commit message: Update

File: urdf/amr.urdf.xacro (robot description, xacro)
@@ -23,5 +23,5 @@
         <parent link="base_footprint"/> <!-- 连接到 base_footprint -->
         <child link="base_link"/> <!-- base_link 作为子链接 -->
-        <origin xyz="0 0 0" rpy="0 0 0"/> <!-- 原点和旋转设置 -->
+        <origin xyz="0 0 0" rpy="0 0 ${pi}"/> <!-- 原点和旋转设置 -->
     </joint>
     <!-- 底盘 (base_link) -->

Commit message: Update

File: urdf/amr.urdf.xacro (robot description, xacro)
@@ -217,5 +217,5 @@
         <parent link="base_link"/>
         <child link="laser"/>
-        <origin xyz="-0.2815 0 0.17223265" rpy="0 0 ${pi}"/> <!-- 激光雷达相对于车体的原点和姿态 -->
+        <origin xyz="-0.2815 0 0.17223265" rpy="0 0 0"/> <!-- 激光雷达相对于车体的原点和姿态 -->
     </joint>
 </robot>

Commit message: Update

File: urdf/amr.urdf.xacro (robot description, xacro)
@@ -217,5 +217,5 @@
         <parent link="base_link"/>
         <child link="laser"/>
-        <origin xyz="-0.2815 0 0.17223265" rpy="0 0 0"/> <!-- 激光雷达相对于车体的原点和姿态 -->
+        <origin xyz="0.2815 0 0.17223265" rpy="0 0 ${pi}"/> <!-- 激光雷达相对于车体的原点和姿态 -->
     </joint>
 </robot>

Commit message: Update

File: urdf/amr.urdf.xacro (robot description, xacro)
@@ -23,5 +23,5 @@
         <parent link="base_footprint"/> <!-- 连接到 base_footprint -->
         <child link="base_link"/> <!-- base_link 作为子链接 -->
-        <origin xyz="0 0 0" rpy="0 0 ${pi}"/> <!-- 原点和旋转设置 -->
+        <origin xyz="0 0 0" rpy="0 0 0"/> <!-- 原点和旋转设置 -->
     </joint>
     <!-- 底盘 (base_link) -->

Commit message: Update

File: urdf/amr.urdf.xacro (robot description, xacro)
@@ -9,4 +9,5 @@
     <xacro:property name="caster_color" value="0.0 0.0 0.0 1.0"/> <!-- 前后万向轮的颜色：黑色 -->
     <xacro:property name="lidar_color" value="0.0 0.0 0.0 1.0"/> <!-- 激光雷达的颜色：黑色 -->
+    <xacro:property name="imu_color" value="0.0 0.0 1.0 1.0"/> <!-- 惯性测量单元的颜色：蓝色 -->
     <!-- 虚拟根链接 (base_footprint) -->
     <!-- base_footprint 是虚拟的参考框架，用来定义机器人在地面上的位置和姿态 -->
@@ -219,3 +220,32 @@
         <origin xyz="0.2815 0 0.17223265" rpy="0 0 ${pi}"/> <!-- 激光雷达相对于车体的原点和姿态 -->
     </joint>
+    <!-- 惯性测量单元 (imu) -->
+    <!--
+        参数说明:
+            - 长度: 7.5厘米
+            - 宽度: 6.5厘米
+            - 高度: 1.5厘米
+    -->
+    <link name="imu">
+        <visual>
+            <origin xyz="0 0 0"/>
+            <geometry>
+                <box size="0.075 0.065 0.015"/>  <!-- 设定IMU的尺寸，单位为米 -->
+            </geometry>
+            <material name="blue">
+                <color rgba="${imu_color}"/>
+            </material>
+        </visual>
+        <collision>
+            <geometry>
+                <box size="0.075 0.065 0.015"/>
+            </geometry>
+        </collision>
+    </link>
+    <!-- imu 通过固定关节连接到 base_link -->
+    <joint name="base_link_to_imu" type="fixed">
+        <parent link="base_link"/>
+        <child link="laser"/>
+        <origin xyz="0.2575 0.1025 0.015" rpy="0 0 0"/> <!-- 激光雷达相对于车体的原点和姿态 -->
+    </joint>
 </robot>

Commit message: Update

File: urdf/amr.urdf.xacro (robot description, xacro)
@@ -246,5 +246,5 @@
     <joint name="base_link_to_imu" type="fixed">
         <parent link="base_link"/>
-        <child link="laser"/>
+        <child link="imu"/>
         <origin xyz="0.2575 0.1025 0.015" rpy="0 0 0"/> <!-- 激光雷达相对于车体的原点和姿态 -->
     </joint>

Commit message: Update

File: urdf/amr.urdf.xacro (robot description, xacro)
@@ -247,5 +247,5 @@
         <parent link="base_link"/>
         <child link="imu"/>
-        <origin xyz="0.2575 0.1025 0.015" rpy="0 0 0"/> <!-- 激光雷达相对于车体的原点和姿态 -->
+        <origin xyz="0.2575 0.1025 0.035" rpy="0 0 0"/> <!-- 激光雷达相对于车体的原点和姿态 -->
     </joint>
 </robot>

Commit message: update

File: urdf/amr.urdf.xacro (robot description, xacro)
@@ -24,5 +24,5 @@
         <parent link="base_footprint"/> <!-- 连接到 base_footprint -->
         <child link="base_link"/> <!-- base_link 作为子链接 -->
-        <origin xyz="0 0 0" rpy="0 0 0"/> <!-- 原点和旋转设置 -->
+        <origin xyz="0 0 0.02" rpy="0 0 0"/> <!-- 原点和旋转设置 -->
     </joint>
     <!-- 底盘 (base_link) -->
@@ -36,5 +36,5 @@
     <link name="base_link">
         <visual>
-            <origin xyz="0 0 0.02" rpy="0 0 0" />
+            <origin xyz="0 0 0" rpy="0 0 0" />
             <geometry>
                 <!-- 视觉形状 -->
@@ -220,32 +220,2 @@
         <origin xyz="0.2815 0 0.17223265" rpy="0 0 ${pi}"/> <!-- 激光雷达相对于车体的原点和姿态 -->
     </joint>
-    <!-- 惯性测量单元 (imu) -->
-    <!--
-        参数说明:
-            - 长度: 7.5厘米
-            - 宽度: 6.5厘米
-            - 高度: 1.5厘米
-    -->
-    <link name="imu">
-        <visual>
-            <origin xyz="0 0 0"/>
-            <geometry>
-                <box size="0.075 0.065 0.015"/>  <!-- 设定IMU的尺寸，单位为米 -->
-            </geometry>
-            <material name="blue">
-                <color rgba="${imu_color}"/>
-            </material>
-        </visual>
-        <collision>
-            <geometry>
-                <box size="0.075 0.065 0.015"/>
-            </geometry>
-        </collision>
-    </link>
-    <!-- imu 通过固定关节连接到 base_link -->
-    <joint name="base_link_to_imu" type="fixed">
-        <parent link="base_link"/>
-        <child link="imu"/>
-        <origin xyz="0.2575 0.1025 0.035" rpy="0 0 0"/> <!-- 激光雷达相对于车体的原点和姿态 -->
-    </joint>
-</robot>

Commit message: update

File: urdf/amr.urdf.xacro (robot description, xacro)
@@ -9,5 +9,4 @@
     <xacro:property name="caster_color" value="0.0 0.0 0.0 1.0"/> <!-- 前后万向轮的颜色：黑色 -->
     <xacro:property name="lidar_color" value="0.0 0.0 0.0 1.0"/> <!-- 激光雷达的颜色：黑色 -->
-    <xacro:property name="imu_color" value="0.0 0.0 1.0 1.0"/> <!-- 惯性测量单元的颜色：蓝色 -->
     <!-- 虚拟根链接 (base_footprint) -->
     <!-- base_footprint 是虚拟的参考框架，用来定义机器人在地面上的位置和姿态 -->

Commit message: update

File: urdf/amr.urdf.xacro (robot description, xacro)
@@ -13,5 +13,5 @@
     <link name="base_footprint">
         <visual>
-            <origin xyz="0 0 0" rpy="0 0 0" />
+            <origin xyz="0 0 0.02" rpy="0 0 0" />
             <geometry>
                 <box size="0.05 0.05 0.001" />

Commit message: update

File: urdf/amr.urdf.xacro (robot description, xacro)
@@ -13,5 +13,5 @@
     <link name="base_footprint">
         <visual>
-            <origin xyz="0 0 0.02" rpy="0 0 0" />
+            <origin xyz="0 0 0" rpy="0 0 0" />
             <geometry>
                 <box size="0.05 0.05 0.001" />
@@ -23,5 +23,5 @@
         <parent link="base_footprint"/> <!-- 连接到 base_footprint -->
         <child link="base_link"/> <!-- base_link 作为子链接 -->
-        <origin xyz="0 0 0.02" rpy="0 0 0"/> <!-- 原点和旋转设置 -->
+        <origin xyz="0 0 0" rpy="0 0 0"/> <!-- 原点和旋转设置 -->
     </joint>
     <!-- 底盘 (base_link) -->
@@ -35,5 +35,5 @@
     <link name="base_link">
         <visual>
-            <origin xyz="0 0 0" rpy="0 0 0" />
+            <origin xyz="0 0 0.02" rpy="0 0 0" />
             <geometry>
                 <!-- 视觉形状 -->

Commit message: update

File: urdf/amr.urdf.xacro (robot description, xacro)
@@ -23,5 +23,5 @@
         <parent link="base_footprint"/> <!-- 连接到 base_footprint -->
         <child link="base_link"/> <!-- base_link 作为子链接 -->
-        <origin xyz="0 0 0" rpy="0 0 0"/> <!-- 原点和旋转设置 -->
+        <origin xyz="0 0 -0.02" rpy="0 0 0"/> <!-- 原点和旋转设置 -->
     </joint>
     <!-- 底盘 (base_link) -->
@@ -35,5 +35,5 @@
     <link name="base_link">
         <visual>
-            <origin xyz="0 0 0.02" rpy="0 0 0" />
+            <origin xyz="0 0 0" rpy="0 0 0" />
             <geometry>
                 <!-- 视觉形状 -->

Commit message: update

File: urdf/amr.urdf.xacro (robot description, xacro)
@@ -23,5 +23,5 @@
         <parent link="base_footprint"/> <!-- 连接到 base_footprint -->
         <child link="base_link"/> <!-- base_link 作为子链接 -->
-        <origin xyz="0 0 -0.02" rpy="0 0 0"/> <!-- 原点和旋转设置 -->
+        <origin xyz="0 0 0.02" rpy="0 0 0"/> <!-- 原点和旋转设置 -->
     </joint>
     <!-- 底盘 (base_link) -->

Commit message: update

File: urdf/amr.urdf.xacro (robot description, xacro)
@@ -217,5 +217,5 @@
         <parent link="base_link"/>
         <child link="laser"/>
-        <origin xyz="0.2815 0 0.17223265" rpy="0 0 ${pi}"/> <!-- 激光雷达相对于车体的原点和姿态 -->
+        <origin xyz="0.2815 0 0.15223265" rpy="0 0 ${pi}"/> <!-- 激光雷达相对于车体的原点和姿态 -->
     </joint>
 </robot>

Commit message: update

File: urdf/amr.urdf.xacro (robot description, xacro)
@@ -217,5 +217,5 @@
         <parent link="base_link"/>
         <child link="laser"/>
-        <origin xyz="0.2815 0 0.15223265" rpy="0 0 ${pi}"/> <!-- 激光雷达相对于车体的原点和姿态 -->
+        <origin xyz="0.2815 0 0.17223265" rpy="0 0 ${pi}"/> <!-- 激光雷达相对于车体的原点和姿态 -->
     </joint>
 </robot>

Commit message: update

File: urdf/amr.urdf.xacro (robot description, xacro)
@@ -78,5 +78,5 @@
         <parent link="base_link" />
         <child link="left_wheel" />
-        <origin xyz="0 0.23215 0.09"/> <!-- 根据底盘和轮子尺寸设置左轮的位置和离地距离 -->
+        <origin xyz="0 0.23215 0.07"/> <!-- 根据底盘和轮子尺寸设置左轮的位置和离地距离 -->
         <axis xyz="0 1 0" /> <!-- 左轮沿 y 轴旋转 -->
     </joint>
@@ -99,5 +99,5 @@
         <parent link="base_link" />
         <child link="right_wheel" />
-        <origin xyz="0 -0.23215 0.09"/>
+        <origin xyz="0 -0.23215 0.07"/>
         <axis xyz="0 1 0" /> <!-- 右轮沿 y 轴旋转 -->
     </joint>
@@ -120,5 +120,5 @@
         <parent link="base_link"/> <!-- 父链接为车体 -->
         <child link="front_fork"/> <!-- 子链接为叉架 -->
-        <origin xyz="0.264 0 0.0399" rpy="0 0 0"/> <!-- 叉架相对于车体的原点和姿态 -->
+        <origin xyz="0.264 0 0.0169" rpy="0 0 0"/> <!-- 叉架相对于车体的原点和姿态 -->
         <axis xyz="0 0 1"/> <!-- 允许叉架围绕 Z 轴自由旋转（万向功能） -->
     </joint>
@@ -139,5 +139,5 @@
         <parent link="base_link"/> <!-- 父链接为车体 -->
         <child link="back_fork"/> <!-- 子链接为叉架 -->
-        <origin xyz="-0.264 0 0.0399" rpy="0 0 0"/> <!-- 叉架相对于车体的原点和姿态 -->
+        <origin xyz="-0.264 0 0.0169" rpy="0 0 0"/> <!-- 叉架相对于车体的原点和姿态 -->
         <axis xyz="0 0 1"/> <!-- 允许叉架围绕 Z 轴自由旋转（万向功能） -->
     </joint>
@@ -167,5 +167,5 @@
         <parent link="front_fork" />
         <child link="front_caster" />
-        <origin xyz="-0.012 0 -0.0239"/> <!-- 前万向轮放置在底盘前部，离地适中 -->
+        <origin xyz="-0.012 0 -0.0209"/> <!-- 前万向轮放置在底盘前部，离地适中 -->
         <axis xyz="0 1 0"/> <!-- 前万向轮自由旋转 -->
     </joint>
@@ -188,5 +188,5 @@
         <parent link="back_fork" />
         <child link="back_caster" />
-        <origin xyz="-0.012 0 -0.0239"/> <!-- 后万向轮放置在底盘后部，对称于前万向轮 -->
+        <origin xyz="-0.012 0 -0.0209"/> <!-- 后万向轮放置在底盘后部，对称于前万向轮 -->
         <axis xyz="0 1 0"/> <!-- 后万向轮自由旋转 -->
     </joint>
@@ -217,5 +217,5 @@
         <parent link="base_link"/>
         <child link="laser"/>
-        <origin xyz="0.2815 0 0.17223265" rpy="0 0 ${pi}"/> <!-- 激光雷达相对于车体的原点和姿态 -->
+        <origin xyz="0.2815 0 0.15223265" rpy="0 0 ${pi}"/> <!-- 激光雷达相对于车体的原点和姿态 -->
     </joint>
 </robot>

Commit message: update

File: urdf/amr.urdf.xacro (robot description, xacro)
@@ -78,5 +78,5 @@
         <parent link="base_link" />
         <child link="left_wheel" />
-        <origin xyz="0 0.23215 0.07"/> <!-- 根据底盘和轮子尺寸设置左轮的位置和离地距离 -->
+        <origin xyz="0 0.23215 0.09"/> <!-- 根据底盘和轮子尺寸设置左轮的位置和离地距离 -->
         <axis xyz="0 1 0" /> <!-- 左轮沿 y 轴旋转 -->
     </joint>
@@ -99,5 +99,5 @@
         <parent link="base_link" />
         <child link="right_wheel" />
-        <origin xyz="0 -0.23215 0.07"/>
+        <origin xyz="0 -0.23215 0.09"/>
         <axis xyz="0 1 0" /> <!-- 右轮沿 y 轴旋转 -->
     </joint>
@@ -120,5 +120,5 @@
         <parent link="base_link"/> <!-- 父链接为车体 -->
         <child link="front_fork"/> <!-- 子链接为叉架 -->
-        <origin xyz="0.264 0 0.0169" rpy="0 0 0"/> <!-- 叉架相对于车体的原点和姿态 -->
+        <origin xyz="0.264 0 0.0369" rpy="0 0 0"/> <!-- 叉架相对于车体的原点和姿态 -->
         <axis xyz="0 0 1"/> <!-- 允许叉架围绕 Z 轴自由旋转（万向功能） -->
     </joint>
@@ -139,5 +139,5 @@
         <parent link="base_link"/> <!-- 父链接为车体 -->
         <child link="back_fork"/> <!-- 子链接为叉架 -->
-        <origin xyz="-0.264 0 0.0169" rpy="0 0 0"/> <!-- 叉架相对于车体的原点和姿态 -->
+        <origin xyz="-0.264 0 0.0369" rpy="0 0 0"/> <!-- 叉架相对于车体的原点和姿态 -->
         <axis xyz="0 0 1"/> <!-- 允许叉架围绕 Z 轴自由旋转（万向功能） -->
     </joint>
@@ -167,5 +167,5 @@
         <parent link="front_fork" />
         <child link="front_caster" />
-        <origin xyz="-0.012 0 -0.0209"/> <!-- 前万向轮放置在底盘前部，离地适中 -->
+        <origin xyz="-0.012 0 -0.0009"/> <!-- 前万向轮放置在底盘前部，离地适中 -->
         <axis xyz="0 1 0"/> <!-- 前万向轮自由旋转 -->
     </joint>
@@ -188,5 +188,5 @@
         <parent link="back_fork" />
         <child link="back_caster" />
-        <origin xyz="-0.012 0 -0.0209"/> <!-- 后万向轮放置在底盘后部，对称于前万向轮 -->
+        <origin xyz="-0.012 0 -0.0009"/> <!-- 后万向轮放置在底盘后部，对称于前万向轮 -->
         <axis xyz="0 1 0"/> <!-- 后万向轮自由旋转 -->
     </joint>
@@ -217,5 +217,5 @@
         <parent link="base_link"/>
         <child link="laser"/>
-        <origin xyz="0.2815 0 0.15223265" rpy="0 0 ${pi}"/> <!-- 激光雷达相对于车体的原点和姿态 -->
+        <origin xyz="0.2815 0 0.17223265" rpy="0 0 ${pi}"/> <!-- 激光雷达相对于车体的原点和姿态 -->
     </joint>
 </robot>

Commit message: update

File: urdf/amr.urdf.xacro (robot description, xacro)
@@ -167,5 +167,5 @@
         <parent link="front_fork" />
         <child link="front_caster" />
-        <origin xyz="-0.012 0 -0.0009"/> <!-- 前万向轮放置在底盘前部，离地适中 -->
+        <origin xyz="-0.012 0 -0.0209"/> <!-- 前万向轮放置在底盘前部，离地适中 -->
         <axis xyz="0 1 0"/> <!-- 前万向轮自由旋转 -->
     </joint>
@@ -188,5 +188,5 @@
         <parent link="back_fork" />
         <child link="back_caster" />
-        <origin xyz="-0.012 0 -0.0009"/> <!-- 后万向轮放置在底盘后部，对称于前万向轮 -->
+        <origin xyz="-0.012 0 -0.0209"/> <!-- 后万向轮放置在底盘后部，对称于前万向轮 -->
         <axis xyz="0 1 0"/> <!-- 后万向轮自由旋转 -->
     </joint>

Commit message: update

File: urdf/amr.urdf.xacro (robot description, xacro)
@@ -23,5 +23,5 @@
         <parent link="base_footprint"/> <!-- 连接到 base_footprint -->
         <child link="base_link"/> <!-- base_link 作为子链接 -->
-        <origin xyz="0 0 0.02" rpy="0 0 0"/> <!-- 原点和旋转设置 -->
+        <origin xyz="0 0 0" rpy="0 0 0"/> <!-- 原点和旋转设置 -->
     </joint>
     <!-- 底盘 (base_link) -->

Commit message: update

File: urdf/amr.urdf.xacro (robot description, xacro)
@@ -23,5 +23,5 @@
         <parent link="base_footprint"/> <!-- 连接到 base_footprint -->
         <child link="base_link"/> <!-- base_link 作为子链接 -->
-        <origin xyz="0 0 0" rpy="0 0 0"/> <!-- 原点和旋转设置 -->
+        <origin xyz="0 0 0.04" rpy="0 0 0"/> <!-- 原点和旋转设置 -->
     </joint>
     <!-- 底盘 (base_link) -->

Commit message: update

File: urdf/amr.urdf.xacro (robot description, xacro)
@@ -23,5 +23,5 @@
         <parent link="base_footprint"/> <!-- 连接到 base_footprint -->
         <child link="base_link"/> <!-- base_link 作为子链接 -->
-        <origin xyz="0 0 0.04" rpy="0 0 0"/> <!-- 原点和旋转设置 -->
+        <origin xyz="0 0 0.02" rpy="0 0 0"/> <!-- 原点和旋转设置 -->
     </joint>
     <!-- 底盘 (base_link) -->

Commit message: update

File: urdf/amr.urdf.xacro (robot description, xacro)
@@ -223,5 +223,5 @@
         <parent link="base_link"/>
         <child link="laser"/>
-        <origin xyz="0.2815 0 0.17223265" rpy="0 0 ${pi}"/> <!-- 激光雷达相对于车体的原点和姿态 -->
+        <origin xyz="0.2815 0 0.17223265" rpy="0 0 0"/> <!-- 激光雷达相对于车体的原点和姿态 -->
     </joint>
 </robot>

Commit message: update

File: urdf/amr.urdf.xacro (robot description, xacro)
@@ -223,5 +223,5 @@
         <parent link="base_link"/>
         <child link="laser"/>
-        <origin xyz="0.2815 0 0.17223265" rpy="0 0 0"/> <!-- 激光雷达相对于车体的原点和姿态 -->
+        <origin xyz="0.2815 0 0.17223265" rpy="${pi} 0 ${pi}"/> <!-- 激光雷达相对于车体的原点和姿态 -->
     </joint>
 </robot>

Commit message: update

File: urdf/amr.urdf.xacro (robot description, xacro)
@@ -223,5 +223,5 @@
         <parent link="base_link"/>
         <child link="laser"/>
-        <origin xyz="0.2815 0 0.17223265" rpy="${pi} 0 ${pi}"/> <!-- 激光雷达相对于车体的原点和姿态 -->
+        <origin xyz="0.2815 0 0.17223265" rpy="0 0 ${pi}"/> <!-- 激光雷达相对于车体的原点和姿态 -->
     </joint>
 </robot>

Commit message: update

File: urdf/amr.urdf.xacro (robot description, xacro)
@@ -23,5 +23,5 @@
         <parent link="base_footprint"/> <!-- 连接到 base_footprint -->
         <child link="base_link"/> <!-- base_link 作为子链接 -->
-        <origin xyz="0 0 0.02" rpy="0 0 0"/> <!-- 原点和旋转设置 -->
+        <origin xyz="0 0 0.02" rpy="0 0 ${pi}"/> <!-- 原点和旋转设置 -->
     </joint>
     <!-- 底盘 (base_link) -->
