Commit message: update

File: urdf/amr.urdf.xacro (robot description, xacro)
@@ -23,5 +23,5 @@
         <parent link="base_footprint"/> <!-- 连接到 base_footprint -->
         <child link="base_link"/> <!-- base_link 作为子链接 -->
-        <origin xyz="0 0 0.02" rpy="0 0 ${pi}"/> <!-- 原点和旋转设置 -->
+        <origin xyz="0 0 0.02" rpy="0 0 0"/> <!-- 原点和旋转设置 -->
     </joint>
     <!-- 底盘 (base_link) -->

Commit message: update

File: urdf/amr.urdf.xacro (robot description, xacro)
@@ -223,5 +223,5 @@
         <parent link="base_link"/>
         <child link="laser"/>
-        <origin xyz="0.2815 0 0.17223265" rpy="0 0 ${pi}"/> <!-- 激光雷达相对于车体的原点和姿态 -->
+        <origin xyz="0.2815 0 0.17223265" rpy="${pi} ${pi} 0"/> <!-- 激光雷达相对于车体的原点和姿态 -->
     </joint>
 </robot>

Commit message: update

File: urdf/amr.urdf.xacro (robot description, xacro)
@@ -223,5 +223,5 @@
         <parent link="base_link"/>
         <child link="laser"/>
-        <origin xyz="0.2815 0 0.17223265" rpy="${pi} ${pi} 0"/> <!-- 激光雷达相对于车体的原点和姿态 -->
+        <origin xyz="0.2815 0 0.17223265" rpy="0 0 ${pi}"/> <!-- 激光雷达相对于车体的原点和姿态 -->
     </joint>
 </robot>

Commit message: update

File: urdf/amr.urdf.xacro (robot description, xacro)
@@ -78,5 +78,5 @@
         <parent link="base_link" />
         <child link="left_wheel" />
-        <origin xyz="0 0.23215 0.09"/> <!-- 根据底盘和轮子尺寸设置左轮的位置和离地距离 -->
+        <origin xyz="0 -0.23215 0.09"/> <!-- 根据底盘和轮子尺寸设置左轮的位置和离地距离 -->
         <axis xyz="0 1 0" /> <!-- 左轮沿 y 轴旋转 -->
     </joint>
@@ -99,5 +99,5 @@
         <parent link="base_link" />
         <child link="right_wheel" />
-        <origin xyz="0 -0.23215 0.09"/>
+        <origin xyz="0 0.23215 0.09"/>
         <axis xyz="0 1 0" /> <!-- 右轮沿 y 轴旋转 -->
     </joint>

Commit message: update

File: urdf/amr.urdf.xacro (robot description, xacro)
@@ -78,5 +78,5 @@
         <parent link="base_link" />
         <child link="left_wheel" />
-        <origin xyz="0 -0.23215 0.09"/> <!-- 根据底盘和轮子尺寸设置左轮的位置和离地距离 -->
+        <origin xyz="0 0.23215 0.09"/> <!-- 根据底盘和轮子尺寸设置左轮的位置和离地距离 -->
         <axis xyz="0 1 0" /> <!-- 左轮沿 y 轴旋转 -->
     </joint>
@@ -99,5 +99,5 @@
         <parent link="base_link" />
         <child link="right_wheel" />
-        <origin xyz="0 0.23215 0.09"/>
+        <origin xyz="0 -0.23215 0.09"/>
         <axis xyz="0 1 0" /> <!-- 右轮沿 y 轴旋转 -->
     </joint>

Commit message: update

File: urdf/amr.urdf.xacro (robot description, xacro)
@@ -9,4 +9,5 @@
     <xacro:property name="caster_color" value="0.0 0.0 0.0 1.0"/> <!-- 前后万向轮的颜色：黑色 -->
     <xacro:property name="lidar_color" value="0.0 0.0 0.0 1.0"/> <!-- 激光雷达的颜色：黑色 -->
+    <xacro:property name="imu_color" value="0.0 1.0 0.0 1.0"/> <!-- 激光雷达的颜色：绿色 -->
     <!-- 虚拟根链接 (base_footprint) -->
     <!-- base_footprint 是虚拟的参考框架，用来定义机器人在地面上的位置和姿态 -->
@@ -225,3 +226,29 @@
         <origin xyz="0.2815 0 0.17223265" rpy="0 0 ${pi}"/> <!-- 激光雷达相对于车体的原点和姿态 -->
     </joint>
+    <!-- 惯性测量单元 (imu) -->
+    <!--
+        参数说明:
+            - STL 网格文件: imu_link.stl
+    -->
+    <link name="imu_link">
+        <visual>
+            <geometry>
+                <mesh filename="package://amr_description/meshes/imu_link.stl" scale="${stl_scale}"/>
+            </geometry>
+            <material name="green">
+                <color rgba="${imu_color}"/>
+            </material>
+        </visual>
+        <collision>
+            <geometry>
+                <mesh filename="package://amr_description/meshes/imu_link.stl" scale="${stl_scale}"/>
+            </geometry>
+        </collision>
+    </link>
+    <!-- imu 通过固定关节连接到 base_link -->
+    <joint name="base_link_to_imu" type="fixed">
+        <parent link="base_link"/>
+        <child link="imu_link"/>
+        <origin xyz="0.2575 0.1025 0.035" rpy="0 0 0"/>
+    </joint>
 </robot>
